File: 555_Badge/555_Badge.sch (KiCad schematic (older format))
At the start: 15 parts

Commit message: Associate footprints and generate netlist
Parts:
- C1: renamed from C?; footprint (none) -> Capacitor_THT:CP_Radial_D5.0mm_P2.00mm
- C2: renamed from C?; footprint (none) -> Capacitor_THT:CP_Radial_D6.3mm_P2.50mm
- D1, D2: renamed from D?; footprint (none) -> LED_THT:LED_D3.0mm
- Q1: renamed from Q?; footprint Package_TO_SOT_THT:TO-92_Inline -> digikey-footprints:TO-92-3
- R1, R2, R3, R4, R5, R6, R7: renamed from R?; footprint (none) -> Resistor_THT:R_Axial_DIN0207_L6.3mm_D2.5mm_P7.62mm_Horizontal
- U1: renamed from U?; footprint (none) -> 555_Badge:ICM7555-PDIP
- gave numbers to parts that had none: 2
Other:
- moved on the sheet: BAT1, C1, C2, D1, D2, Q1, R1, R2, R3, R4, R5, R6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
